Commit message: added lidar

File: alphabot_base_description/urdf/alphabot_base.xacro (robot description, xacro)
@@ -4,10 +4,9 @@
 <xacro:include filename="$(find alphabot_base_description)/urdf/alphabot_base.trans" />
 <xacro:include filename="$(find alphabot_base_description)/urdf/alphabot_base.gazebo" />
-<!-- <xacro:include filename="$(find alphabot_base_description)/gazebo/alphabot_base_plugins.gazebo" /> -->
 <link name="base_link">
   <inertial>
-    <origin xyz="0.10955796271120455 0.00244443549563504 0.04154096131754149" rpy="0 0 0"/>
-    <mass value="2.0054173190533096"/>
-    <inertia ixx="0.002691" iyy="0.005622" izz="0.006954" ixy="-2.9e-05" iyz="1e-06" ixz="9.6e-05"/>
+    <origin xyz="0.1088047853412877 0.0024273001725789323 0.04130382014186731" rpy="0 0 0"/>
+    <mass value="2.0312240853373598"/>
+    <inertia ixx="0.002725" iyy="0.0058" izz="0.007112" ixy="-3e-05" iyz="1e-06" ixz="3.9e-05"/>
   </inertial>
   <visual>
@@ -25,8 +24,8 @@
   </collision>
 </link>
-<link name="tyre_left_2">
+<link name="tyre_left_2_1">
   <inertial>
-    <origin xyz="-1.0291917068583345e-08 -0.015890267820055454 5.6733905702544e-07" rpy="0 0 0"/>
-    <mass value="0.233413023744858"/>
+    <origin xyz="-1.0294736729754561e-08 -0.01589026768426134 5.673710496145734e-07" rpy="0 0 0"/>
+    <mass value="0.23341302374485776"/>
     <inertia ixx="9.6e-05" iyy="0.00016" izz="9.6e-05" ixy="-0.0" iyz="0.0" ixz="0.0"/>
   </inertial>
@@ -34,5 +33,5 @@
     <origin xyz="-0.13535 0.055077 -0.031954" rpy="0 0 0"/>
     <geometry>
-      <mesh filename="package://alphabot_base_description/meshes/tyre_left_2.stl" scale="0.001 0.001 0.001"/>
+      <mesh filename="package://alphabot_base_description/meshes/tyre_left_2_1.stl" scale="0.001 0.001 0.001"/>
     </geometry>
     <material name="silver"/>
@@ -41,12 +40,12 @@
     <origin xyz="-0.13535 0.055077 -0.031954" rpy="0 0 0"/>
     <geometry>
-      <mesh filename="package://alphabot_base_description/meshes/tyre_left_2.stl" scale="0.001 0.001 0.001"/>
+      <mesh filename="package://alphabot_base_description/meshes/tyre_left_2_1.stl" scale="0.001 0.001 0.001"/>
     </geometry>
   </collision>
 </link>
-<link name="tyre_right_2">
+<link name="tyre_right_2_1">
   <inertial>
-    <origin xyz="-6.416216058457991e-09 0.015890269546393103 5.80426184441929e-07" rpy="0 0 0"/>
-    <mass value="0.23341258097957676"/>
+    <origin xyz="-6.4190364690297486e-09 0.01589026924972143 5.804581818188992e-07" rpy="0 0 0"/>
+    <mass value="0.23341258097957548"/>
     <inertia ixx="9.6e-05" iyy="0.00016" izz="9.6e-05" ixy="0.0" iyz="-0.0" ixz="0.0"/>
   </inertial>
@@ -54,5 +53,5 @@
     <origin xyz="-0.13535 -0.059077 -0.031954" rpy="0 0 0"/>
     <geometry>
-      <mesh filename="package://alphabot_base_description/meshes/tyre_right_2.stl" scale="0.001 0.001 0.001"/>
+      <mesh filename="package://alphabot_base_description/meshes/tyre_right_2_1.stl" scale="0.001 0.001 0.001"/>
     </geometry>
     <material name="silver"/>
@@ -61,19 +60,44 @@
     <origin xyz="-0.13535 -0.059077 -0.031954" rpy="0 0 0"/>
     <geometry>
-      <mesh filename="package://alphabot_base_description/meshes/tyre_right_2.stl" scale="0.001 0.001 0.001"/>
+      <mesh filename="package://alphabot_base_description/meshes/tyre_right_2_1.stl" scale="0.001 0.001 0.001"/>
     </geometry>
   </collision>
 </link>
-<joint name="left_joint" type="continuous">
+<link name="rplidar_1">
+  <inertial>
+    <origin xyz="0.027907600567433848 -0.034766238863451364 0.03526812773284048" rpy="0 0 0"/>
+    <mass value="1.3392997077576572"/>
+    <inertia ixx="0.000967" iyy="0.000619" izz="0.001105" ixy="1e-06" iyz="-0.000159" ixz="-3e-06"/>
+  </inertial>
+  <visual>
+    <origin xyz="-0.028925 -0.03911 -0.07484" rpy="0 0 0"/>
+    <geometry>
+      <mesh filename="package://alphabot_base_description/meshes/rplidar_1.stl" scale="0.001 0.001 0.001"/>
+    </geometry>
+    <material name="silver"/>
+  </visual>
+  <collision>
+    <origin xyz="-0.028925 -0.03911 -0.07484" rpy="0 0 0"/>
+    <geometry>
+      <mesh filename="package://alphabot_base_description/meshes/rplidar_1.stl" scale="0.001 0.001 0.001"/>
+    </geometry>
+  </collision>
+</link>
+<joint name="Rev32" type="continuous">
   <origin xyz="0.13535 -0.055077 0.031954" rpy="0 0 0"/>
   <parent link="base_link"/>
-  <child link="tyre_left_2"/>
+  <child link="tyre_left_2_1"/>
   <axis xyz="0.0 1.0 -0.0"/>
 </joint>
-<joint name="right_joint" type="continuous">
+<joint name="Rev33" type="continuous">
   <origin xyz="0.13535 0.059077 0.031954" rpy="0 0 0"/>
   <parent link="base_link"/>
-  <child link="tyre_right_2"/>
-  <axis xyz="0.0 -1.0 -0.0"/>
+  <child link="tyre_right_2_1"/>
+  <axis xyz="-0.0 1.0 0.0"/>
+</joint>
+<joint name="Rigid34" type="fixed">
+  <origin xyz="0.028925 0.03911 0.07484" rpy="0 0 0"/>
+  <parent link="base_link"/>
+  <child link="rplidar_1"/>
 </joint>
 </robot>
